File: hardware/sd-led-card.kicad_pcb (KiCad board)
At the start: 2 copper layers, 24 x 16 mm, 19 parts, among them J1 SD card edge contacts, U1 RP2350A

Commit message: Document SD slot stiffener envelope
Parts:
- removed the DBG at (0.00, 0.00) (x8)
- added DBG (x8): DBG, , B.Cu at (0.00, 0.00)
Other:
- board text added: "MECH: F-side +0.6mm stiffener here"

Commit message: Add functional schematic scaffold
Parts:
- removed DBG (x8): DBG, 
- added DBG1: SWD/debug pads, , B.Cu at (0.00, 0.00)
Other:
- board text removed: "MECH: F-side +0.6mm stiffener here"
