File: hardware/sd-led-card.kicad_sch (KiCad schematic)
At the start: 0 parts

Commit message: Add functional schematic scaffold
Parts:
- added C1: 100n, Capacitor_SMD:C_0402_1005Metric, symbol SDLED:Capacitor
- added C2: 1u, Capacitor_SMD:C_0402_1005Metric, symbol SDLED:Capacitor
- added CT1: Cap touch, SDLED:Cap_Touch_Pad, symbol SDLED:TouchPad
- added D1, D2, D3, D4, D5, D6: side RGB addressable, LED_SMD:LED_RGB_Everlight_EASV3015RGBA0_Horizontal, symbol SDLED:Addressable_Side_RGB
- added DBG1: SWD/debug pads, SDLED:Debug_Robot_Pads_8, symbol SDLED:DebugPads_8
- added J1: SD edge contacts, Connector_Card:SD_Card_Device_16mm_SlotDepth, symbol SDLED:SD_Edge_9Pin
- added U1: RP2350A, Package_DFN_QFN:QFN-60-1EP_7x7mm_P0.4mm_EP3.4x3.4mm, symbol SDLED:RP2350A_QFN60_Min
Connections:
- new net +3V3: C1.1, C2.1, D1.1 (VDD), D2.1 (VDD), D3.1 (VDD), D4.1 (VDD), D5.1 (VDD), D6.1 (VDD), DBG1.4 (3V3), J1.4 (VDD), U1.14 (3V3)
- new net BOOTSEL: DBG1.8 (BOOTSEL)
- new net CAP_TOUCH: CT1.1 (TOUCH), U1.8 (GP7/CAP_TOUCH)
- new net GND: C1.2, C2.2, D1.3 (GND), D2.3 (GND), D3.3 (GND), D4.3 (GND), D5.3 (GND), D6.3 (GND), DBG1.5 (GND), J1.6 (VSS), J1.9 (VSS2), U1.15 (GND)
- new net LED_D0: D1.4 (DIN), U1.7 (GP6/LED_DIN)
- new net LED_D1: D1.2 (DOUT), D2.4 (DIN)
- new net LED_D2: D2.2 (DOUT), D3.4 (DIN)
- new net LED_D3: D3.2 (DOUT), D4.4 (DIN)
- new net LED_D4: D4.2 (DOUT), D5.4 (DIN)
- new net LED_D5: D5.2 (DOUT), D6.4 (DIN)
- new net RUN: DBG1.3 (RUN), U1.11 (RUN)
- new net SD_CLK: J1.5 (CLK), U1.2 (GP1/SD_CLK)
- new net SD_CMD: J1.3 (CMD), U1.1 (GP0/SD_CMD)
- new net SD_DAT0: J1.7 (DAT0), U1.3 (GP2/SD_DAT0)
- new net SD_DAT1: J1.8 (DAT1), U1.4 (GP3/SD_DAT1)
- new net SD_DAT2: J1.1 (DAT2), U1.5 (GP4/SD_DAT2)
- new net SD_DAT3: J1.2 (DAT3/CD), U1.6 (GP5/SD_DAT3)
- new net SWCLK: DBG1.2 (SWCLK), U1.10 (SWCLK)
- new net SWDIO: DBG1.1 (SWDIO), U1.9 (SWDIO)
- new net UART_RX: DBG1.7 (UART_RX), U1.13 (UART_RX)
- new net UART_TX: DBG1.6 (UART_TX), U1.12 (UART_TX)
- no-connect marks 0 -> 46
